File: Kicad/A4092/A4092.kicad_sch (KiCad schematic)
At the start: 0 parts

Commit message: First version of A4770 cheetah
Other:
- sheet CPLD renamed CPLD, Flash & Clock
- sheet SCSI-2 Controller renamed SCSI Host Controller
- sheet Termination & Connectors renamed Termination, Power & Connectors
- removed sheet Caps & Power
- removed sheet Flash memory
- note added: "Advanced UW SCSI Controller Board This Zorro III board is based on the A4091 which was designed and sold by Commodore and DKB Software. Features: • SPI Boot ROM • LSI 53C770 SCSI II controller • 68 pin internal connector • 68 pin external SCSI2 connector • Active SCSI termination • Zorro III bus support Based on the A4091 SCSI2 controller. The Commodore A4091 was reverse-engineered by Stefan Rein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"
- note added: "Amiga Cheetah 4770 UW SCSI Host Controller"
- note added: "GitHub Project: https://github.com/A4091/a4092-dev"
- note removed: "Advanced SCSI II Controller Board This Zorro III board is based on the A4091 which was designed and sold by Commodore and DKB Software. Features: • Boot ROM • NCR 53C710 SCSI II controller • 50 pin internal connector • 50 pin external SCSI2 connector • Active SCSI termination • Zorro III bus support Caveats: • Requires Buster 11 • Does not work with with A3640 Rev 3.0 • No RAM option • No wide SC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"
- note removed: "Amiga 4092 SCSI-2 Host Controller"
- note removed: "GitHub Project: https://github.com/A4091/ Schematics: https://github.com/A4091/a4091-hardware/blob/main/schematics/ReA4091_Rev4_2023-05-15_Schematic.pdf"
- title: A4092 -> Cheetah UW
Changed lines of the file:
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@@
 	(paper "A4")
 	(title_block
-		(title "A4092")
-		(rev "PROTO0")
+		(title "Cheetah UW")
+		(rev "PROTO1")
 		(company "amiga.technology")
 	)
-	(text "Advanced SCSI II Controller Board\nThis Zorro III board is based on the A4091 which was designed and sold by Commodore and\nDKB Software.\nFeatures:\n• Boot ROM\n• NCR 53C710 SCSI II controller\n• 50 pin internal connector\n• 50 pin external SCSI2 connector\n• Active SCSI termination\n• Zorro III bus support\nCaveats:\n• Requires Buster 11\n• Does not work with with A3640 Rev 3.0\n• No RAM option\n• No wide SCSI support\n\nThe Commodore A4091 was reverse-engineered by Stefan Reinauer and Chris Hooper. "
+	(text "Advanced UW SCSI Controller Board\nThis Zorro III board is based on the A4091 which was designed and sold by Commodore and\nDKB Software.\nFeatures:\n• SPI Boot ROM\n• LSI 53C770 SCSI II controller\n• 68 pin internal connector\n• 68 pin external SCSI2 connector\n• Active SCSI termination\n• Zorro III bus support\n\nBased on the A4091 SCSI2 controller. The Commodore A4091 was \nreverse-engineered by Stefan Reinauer and Chris Hooper. "
 		(exclude_from_sim no)
-		(at 51.816 105.156 0)
+		(at 69.596 98.806 0)
 		(effects
 			(font
@@
 		)
 	)
-	(text "GitHub Project:\nhttps://github.com/A4091/\n\nSchematics:\nhttps://github.com/A4091/a4091-hardware/blob/main/schematics/ReA4091_Rev4_2023-05-15_Schematic.pdf"
+	(text "GitHub Project:\nhttps://github.com/A4091/a4092-dev"
 		(exclude_from_sim no)
-		(at 157.734 153.162 0)
+		(at 163.83 141.732 0)
 		(effects
 			(font
@@
 		)
 	)
-	(text "Amiga 4092 SCSI-2 Host Controller\n"
+	(text "Amiga Cheetah 4770 UW SCSI Host Controller\n"
 		(exclude_from_sim no)
-		(at 122.428 64.262 0)
+		(at 159.004 63.754 0)
 		(effects
 			(font
@@
 	)
 	(sheet
-		(at 187.96 21.59)
+		(at 119.38 22.86)
 		(size 35.56 29.21)
 		(exclude_from_sim no)
@@
 			(color 0 0 0 0.0000)
 		)
-		(property "Sheetname" "Caps & Power"
-			(at 187.96 20.8784 0)
-			(effects
-				(font
-					(size 1.27 1.27)
-				)
-				(justify left bottom)
-			)
-		)
-		(property "Sheetfile" "power.kicad_sch"
-			(at 187.96 51.3846 0)
-			(effects
-				(font
-					(size 1.27 1.27)
-				)
-				(justify left top)
-			)
-		)
-		(instances
-			(project "A4092"
-				(path "/8f9f4021-47aa-41d9-bea7-f6ccf72098bb"
-					(page "6")
-				)
-			)
-		)
-	)
-	(sheet
-		(at 73.66 21.59)
-		(size 35.56 29.21)
-		(exclude_from_sim no)
-		(in_bom yes)
-		(on_board yes)
-		(dnp no)
-		(fields_autoplaced yes)
-		(stroke
-			(width 0.1524)
-			(type solid)
-		)
-		(fill
-			(color 0 0 0 0.0000)
-		)
-		(property "Sheetname" "SCSI-2 Controller"
-			(at 73.66 20.8784 0)
+		(property "Sheetname" "SCSI Host Controller"
+			(at 119.38 22.1484 0)
 			(effects
 				(font
@@
 		)
 		(property "Sheetfile" "scsi2.kicad_sch"
-			(at 73.66 51.3846 0)
+			(at 119.38 52.6546 0)
 			(effects
 				(font
@@
 	)
 	(sheet
-		(at 35.56 21.59)
+		(at 81.28 22.86)
 		(size 35.56 29.21)
 		(exclude_from_sim no)
@@
 			(color 0 0 0 0.0000)
 		)
-		(property "Sheetname" "Termination & Connectors"
-			(at 35.56 20.8784 0)
+		(property "Sheetname" "Termination, Power & Connectors"
+			(at 81.28 22.1484 0)
 			(effects
 				(font
@@
 		)
 		(property "Sheetfile" "Termination.kicad_sch"
-			(at 35.56 51.3846 0)
+			(at 81.28 52.6546 0)
 			(effects
 				(font
@@
 	)
 	(sheet
-		(at 111.76 21.59)
+		(at 157.48 22.86)
 		(size 35.56 29.21)
 		(exclude_from_sim no)
@@
 		)
 		(property "Sheetname" "Zorro III bus"
-			(at 111.76 20.8784 0)
+			(at 157.48 22.1484 0)
 			(effects
 				(font
@@
 		)
 		(property "Sheetfile" "zorro3.kicad_sch"
-			(at 111.76 51.3846 0)
+			(at 157.48 52.6546 0)
 			(effects
 				(font
@@
 	)
 	(sheet
-		(at 226.0914 21.5967)
-		(size 35.5286 29.2033)
-		(exclude_from_sim no)
-		(in_bom yes)
-		(on_board yes)
-		(dnp no)
-		(fields_autoplaced yes)
-		(stroke
-			(width 0.1524)
-			(type solid)
-		)
-		(fill
-			(color 0 0 0 0.0000)
-		)
-		(property "Sheetname" "Flash memory"
-			(at 226.0914 20.8851 0)
-			(effects
-				(font
-					(size 1.27 1.27)
-				)
-				(justify left bottom)
-			)
-		)
-		(property "Sheetfile" "flash.kicad_sch"
-			(at 226.0914 51.3846 0)
-			(effects
-				(font
-					(size 1.27 1.27)
-				)
-				(justify left top)
-			)
-		)
-		(instances
-			(project "A4092"
-				(path "/8f9f4021-47aa-41d9-bea7-f6ccf72098bb"
-					(page "7")
-				)
-			)
-		)
-	)
-	(sheet
-		(at 149.86 21.59)
+		(at 195.58 22.86)
 		(size 35.56 29.21)
 		(exclude_from_sim no)
@@
 			(color 0 0 0 0.0000)
 		)
-		(property "Sheetname" "CPLD"
-			(at 149.86 20.8784 0)
+		(property "Sheetname" "CPLD, Flash & Clock"
+			(at 195.58 22.1484 0)
 			(effects
 				(font
@@
 		)
 		(property "Sheetfile" "cpld.kicad_sch"
-			(at 149.86 51.3846 0)
+			(at 195.58 52.6546 0)
 			(effects
 				(font
