File: Kicad/A4092/A4092.kicad_pcb (KiCad board)
At the start: 4 copper layers, 175.6 x 96.4 mm, 127 parts, among them CN1 Zorro3, J1 5749721-7, J2 5749721-7, J3 TO-LED, J4 TO-MB, J5 TO-A3000-LED, J6 TO-A3000-MB, J8 Conn_01x06_Pin, U1 SN74ABT16543DGGR, U10 DS21S07A, U11 DS21S07A, U12 DS21S07A, U13 W25X40CLSN, U2 SN74ABT16543DGGR, U3 SN74ABT16543DGGR, U4 SN74ABT16543DGGR, U5 74LVC07APW_118, U6 SN74ABT16543DGGR, U7 AMS1117-3.3, U8 XC95144XL-TQ144, U9 LSI53C770 SCSI Host Controller, Y1 Abracon ACO-50MHz, Y2 Abracon ACO-40MHz

Commit message: Routing
Parts:
- moved C80 25.8 mm to (73.0, 99.5), turned to -90 degrees
- moved C96 4.61 mm to (156.5, 98.5), turned to 0 degrees
- moved C85 3.50 mm to (104.0, 92.0), turned to 45 degrees
- moved R96 3.00 mm to (117.0, 98.0)
- moved C97 2.69 mm to (135.5, 78.0), turned to 180 degrees
- moved C91 2.50 mm to (117.0, 96.0), turned to 180 degrees
- moved kibuzzard-696E6D75 1.09 mm to (53.5, 127.5)
- moved R108 1.00 mm to (156.5, 96.0)
Routing:
- net SCSI_TERMPWR: track 89.6 -> 179.0 mm, vias 1 -> 10
- net GND: track 143.4 -> 181.2 mm, vias 273 -> 272
- net PLD_DS: track 71.6 -> 95.1 mm, vias 1 -> 2
- net D15: track 57.4 -> 78.6 mm, vias 1 -> 2
- net V5: track 193.6 -> 214.3 mm, vias 16 -> 24
- net PLD_READ: track 131.6 -> 149.0 mm, vias 4 -> 5
- net LEDR: track 25.0 -> 41.4 mm
- net D0: track 72.3 -> 87.6 mm
- net SCDAT12: track 110.4 -> 125.6 mm, vias 2 -> 5
- net PLD_AS: track 41.0 -> 55.6 mm, vias 1 -> 2
- net V3_3: track 39.2 -> 51.5 mm, vias 3 -> 4
- net NCR_INT: track 67.0 -> 79.1 mm, vias 1 -> 2
- net SREG: track 68.0 -> 76.3 mm, vias 1 -> 2
- net D2Z: track 91.6 -> 95.9 mm, vias 3 -> 5
- net TCK: track 26.7 -> 30.7 mm
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
Commit message: PWR and GND routing
Parts:
- moved R68 3.81 mm to (105.5, 137.5), turned to 0 degrees
- moved C84 3.04 mm to (91.0, 112.0), turned to -45 degrees
- moved C81 0.71 mm to (103.5, 100.5)
Routing:
- net V3_3: track 51.5 -> 224.4 mm, vias 4 -> 18
- net GND: track 181.2 -> 219.4 mm, vias 272 -> 322
- net V5: track 214.3 -> 245.7 mm, vias 24 -> 34
- net PLD_READ: track 149.0 -> 152.3 mm
- net A16: track 87.6 -> 85.4 mm
- net A15: track 118.0 -> 116.2 mm
- net A17: track 133.3 -> 135.0 mm
- net A7: track 130.1 -> 128.5 mm
- net A6: track 130.7 -> 129.0 mm
- net Z_SLAVE: track 156.8 -> 155.4 mm
- net SCLK: track 138.9 -> 140.3 mm
- net SCTRL_CD: track 133.5 -> 134.7 mm
- net SLACK: track 77.5 -> 78.7 mm
- net A4: track 132.4 -> 133.4 mm, vias 5 -> 3
- net A5: track 134.0 -> 134.9 mm, vias 5 -> 3
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