File: Kicad/A4770/A4770.kicad_pcb (KiCad board)
At the start: 4 copper layers, 175.6 x 96.4 mm, 127 parts, among them CN1 Zorro3, J1 5749721-7, J2 5787082-7, J3 TO-LED, J4 TO-MB, J5 TO-A3000-LED, J6 TO-A3000-MB, J8 Conn_01x06_Pin, U1 SN74ABT16543DGGR, U10 DS21S07A, U11 DS21S07A, U12 DS21S07A, U13 W25X40CLSN, U2 SN74ABT16543DGGR, U3 SN74ABT16543DGGR, U4 SN74ABT16543DGGR, U5 74LVC07APW_118, U6 SN74ABT16543DGGR, U7 AMS1117-3.3, U8 XC95144XL-TQ144, U9 LSI53C770 SCSI Host Controller, Y1 Abracon ACO-50MHz, Y2 Abracon ACO-40MHz

Commit message: PWR and GND routing
Parts:
- moved C92 8.86 mm to (125.5, 114.0), turned to -90 degrees
- moved C93 5.50 mm to (131.5, 114.0)
- moved C91 1.80 mm to (118.5, 95.0), turned to 90 degrees
- moved C20 0.50 mm to (131.0, 120.5)
- moved R107 0.50 mm to (134.0, 114.0)
Routing:
- net V5: track 287.5 -> 462.0 mm, vias 37 -> 44
- net D19: track 25.0 -> 19.8 mm
- net RAMCS: track 55.6 -> 51.7 mm
- net A16: track 88.1 -> 91.7 mm
- net Net-(Y2-OUT): track 0.00 -> 3.61 mm
- net D2Z: track 96.9 -> 93.9 mm
- net LED: track 87.2 -> 89.2 mm
- net Net-(R5-Pad2): track 0.00 -> 2.02 mm
- net D25: track 64.6 -> 66.4 mm
- net D31: track 61.6 -> 59.9 mm
- net D24: track 63.1 -> 64.5 mm
- net BCLK: track 58.8 -> 57.7 mm
- net Z_A29D29: track 74.0 -> 73.0 mm
- net GND: track 376.9 -> 377.5 mm, vias 358 -> 363
- net Z_CINH: track 148.6 -> 148.0 mm
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