File: Kicad/A4770/A4770.kicad_pcb (KiCad board)
At the start: 4 copper layers, 175.6 x 96.4 mm, 127 parts, among them CN1 Zorro3, J1 5749721-7, J2 5787082-7, J3 TO-LED, J4 TO-MB, J5 TO-A3000-LED, J6 TO-A3000-MB, J8 Conn_01x06_Pin, U1 SN74ABT16543DGGR, U10 DS21S07A, U11 DS21S07A, U12 DS21S07A, U13 W25X40CLSN, U2 SN74ABT16543DGGR, U3 SN74ABT16543DGGR, U4 SN74ABT16543DGGR, U5 74LVC07APW_118, U6 SN74ABT16543DGGR, U7 AMS1117-3.3, U8 XC95144XL-TQ144, U9 LSI53C770 SCSI Host Controller, Y1 Abracon ACO-50MHz, Y2 Abracon ACO-40MHz

Commit message: Fix up part numbers
Parts:
- D1: value SS24 -> SS34
- D2: value LED (green) -> LED
- J2: value 5787082-7 -> 5749721-7
