File: Kicad/A4770/zorro3.kicad_sch (KiCad schematic)
At the start: 39 parts, among them CN1 Zorro3, U1 SN74ABT16543DGGR, U2 SN74ABT16543DGGR, U3 SN74ABT16543DGGR, U4 SN74ABT16543DGGR, U5 74LVC07APW_118, U6 SN74ABT16543DGGR

Commit message: Fix footprints
Parts:
- U1, U2, U3, U4, U6: footprint DGG56 -> SN74ABT16543DGGR:DGG56
Changed lines of the file:
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@@
 			)
 		)
-		(property "Footprint" "DGG56"
+		(property "Footprint" "SN74ABT16543DGGR:DGG56"
 			(at 125.73 133.35 0)
 			(effects
@@
 			)
 		)
-		(property "Footprint" "DGG56"
+		(property "Footprint" "SN74ABT16543DGGR:DGG56"
 			(at 228.6 31.75 0)
 			(effects
@@
 			)
 		)
-		(property "Footprint" "DGG56"
+		(property "Footprint" "SN74ABT16543DGGR:DGG56"
 			(at 27.94 31.75 0)
 			(effects
@@
 			)
 		)
-		(property "Footprint" "DGG56"
+		(property "Footprint" "SN74ABT16543DGGR:DGG56"
 			(at 27.94 133.35 0)
 			(effects
@@
 			)
 		)
-		(property "Footprint" "DGG56"
+		(property "Footprint" "SN74ABT16543DGGR:DGG56"
 			(at 125.73 30.48 0)
 			(effects
